File: base_board/beer_mug.sch (KiCad schematic (older format))
At the start: 17 parts, among them J1 Conn_ARM_JTAG_SWD_10, J2 Conn_01x02_Female, J3 Conn_01x04_Female, J4 Conn_01x02_Female, J5 Conn_01x03_Female, J6 Conn_01x02_Female, U1 MAX11212, U2 MCP73832-2-OT, U3 Itsy-Bitsy-M0

Commit message: updated schematic
Parts:
- removed J1: Conn_ARM_JTAG_SWD_10, symbol Connector:Conn_ARM_JTAG_SWD_10
- removed J2, J4, J6: Conn_01x02_Female, symbol Connector:Conn_01x02_Female
- removed J3: Conn_01x04_Female, symbol Connector:Conn_01x04_Female
- removed J5: Conn_01x03_Female, symbol Connector:Conn_01x03_Female
- removed U1: MAX11212, beer_mug:uMAX10, symbol beer_mug:MAX11212
- added H1, H2: MountingHole, MountingHole:MountingHole_3.2mm_M3_DIN965_Pad_TopBottom, symbol Mechanical:MountingHole
- added J1, J2, J4, J6: Conn_01x02, Connector_PinHeader_1.27mm:PinHeader_1x02_P1.27mm_Vertical, symbol Connector_Generic:Conn_01x02
- added J3: Conn_01x08, Connector_PinHeader_1.27mm:PinHeader_1x08_P1.27mm_Vertical, symbol Connector_Generic:Conn_01x08
- added J5: Conn_01x03, Connector_PinHeader_1.27mm:PinHeader_1x03_P1.27mm_Vertical, symbol Connector_Generic:Conn_01x03
- added Q7: Q_NMOS_DGS, Package_TO_SOT_SMD:SOT-23, symbol Device:Q_NMOS_DGS
- added R10, R11, R8, R9: R, Resistor_SMD:R_0603_1608Metric, symbol Device:R
- added U1, U4: OPA322, Package_TO_SOT_SMD:SOT-23-5, symbol Amplifier_Operational:OPA330xxDBV
- C1, C2: footprint (none) -> Capacitor_SMD:C_0805_2012Metric
- C3, C4: footprint (none) -> Capacitor_SMD:C_0603_1608Metric
- R13: footprint (none) -> Resistor_SMD:R_0603_1608Metric
- R14: footprint Resistor_THT:R_Axial_DIN0309_L9.0mm_D3.2mm_P12.70mm_Horizontal -> Resistor_SMD:R_0603_1608Metric
Connections:
- net +3V3: now also C4.1, J3.1 (Pin_1), J5.1 (Pin_1), J6.1 (Pin_1), U1.5 (V+), U4.5 (V+); no longer C4.2, U3.3 (AREF)
- net +BATT: now also J2.1 (Pin_1), J3.7 (Pin_7); no longer U3.33 (VBAT)
- net 1Wire: now also U3.19 (D4), J5.3 (Pin_3); no longer U3.27 (D10)
- net AREF: now also U3.3 (AREF), R11.1, U4.3 (+)
- net GND: now also C4.2, J1.2 (Pin_2), J2.2 (Pin_2), J3.2 (Pin_2), J4.2 (Pin_2), J5.2 (Pin_2), R10.2, R9.2, U1.2 (V-), U4.2 (V-); no longer C4.1
- net Green: now also U3.28 (D11); no longer U3.29 (D12)
- net I2C_SCL: now also J3.4 (Pin_4)
- net I2C_SDA: now also J3.3 (Pin_3)
- net Red: now also U3.27 (D10); no longer U3.28 (D11)
- net VBUS: now also J4.1 (Pin_1)
- net A5: now reaches U3.10 (A5)
- net A5: now also R8.1, U1.1
- net Button_1: now reaches U3.21 (D1)
- net Button_1: now also J3.5 (Pin_5)
- net A1: now reaches U3.6 (A1)
- net A1: now also J1.1 (Pin_1), R11.2
- net SPI_MOSI: no longer names the net of U3.13 (MISO)
- net SPI_MOSI: no longer U3.20 (D0)
- net SPI_SCK: no longer names the net of U3.11 (SCK)
- net SWCLK: no longer names the net of U3.17 (SWCLK)
- net SWDIO: no longer names the net of U3.16 (SWDIO)
- net nEN: no longer names the net of U3.15 (EN)
- net nReset: no longer names the net of U3.1 (nRESET)
- new net: R8.2, R9.1, U1.4 (-)
- new net: Q7.2 (G), U4.1
- new net: Q7.3 (S), R10.1, U4.4 (-)
- new net Button_2: J3.6 (Pin_6), U3.20 (D0)
- new net FLUID_SENSE-: J6.2 (Pin_2), Q7.1 (D), U1.3 (+)
- new net VBAT_SWITCHED: J3.8 (Pin_8), U3.33 (VBAT)
Other:
- note added: "Battery"
- note added: "Display / IO"
- note added: "External Supply /\nBattery Charge"
- moved on the sheet: C1, C2, D2, R13, R14, R7, U2
