File: base_board/led_nmos.sch (KiCad schematic (older format))
At the start: 2 parts, among them Q1 Q_NMOS_DGS

Commit message: updated schematic
Parts:
- Q1: footprint (none) -> Package_TO_SOT_SMD:SOT-23
- R1: footprint (none) -> Resistor_SMD:R_0603_1608Metric
Changed lines of the file:
@@
 $Descr A4 11693 8268
 encoding utf-8
-Sheet 4 5
+Sheet 2 5
 Title ""
 Date ""
@@
 F 0 "Q3" H 4855 3046 50  0000 L CNN
 F 1 "Q_NMOS_DGS" H 4855 2955 50  0000 L CNN
-F 2 "" H 4850 3100 50  0001 C CNN
+F 2 "Package_TO_SOT_SMD:SOT-23" H 4850 3100 50  0001 C CNN
 F 3 "~" H 4650 3000 50  0001 C CNN
 	1    4650 3000
@@
 F 0 "R3" H 4620 2596 50  0000 L CNN
 F 1 "R" H 4620 2505 50  0000 L CNN
-F 2 "" V 4480 2550 50  0001 C CNN
+F 2 "Resistor_SMD:R_0603_1608Metric" V 4480 2550 50  0001 C CNN
 F 3 "~" H 4550 2550 50  0001 C CNN
 	1    4550 2550
