File: base_board/rgb_led.sch (KiCad schematic (older format))
At the start: 7 parts, among them Q4 Q_PMOS_DGS, Q5 Q_PMOS_DGS, Q6 Q_PMOS_DGS

Commit message: updated schematic
Parts:
- D1: footprint (none) -> LED_THT:LED_D5.0mm-4_RGB
- Q4, Q5, Q6: footprint (none) -> Package_TO_SOT_SMD:SOT-23
- R4, R5, R6: footprint (none) -> Resistor_SMD:R_0603_1608Metric
Changed lines of the file:
@@
 $Descr A4 11693 8268
 encoding utf-8
-Sheet 5 5
+Sheet 4 5
 Title ""
 Date ""
@@
 F 0 "D1" V 4854 3760 50  0000 L CNN
 F 1 "LED_RAGB" V 4945 3760 50  0000 L CNN
-F 2 "" H 4900 3350 50  0001 C CNN
+F 2 "LED_THT:LED_D5.0mm-4_RGB" H 4900 3350 50  0001 C CNN
 F 3 "~" H 4900 3350 50  0001 C CNN
 	1    4900 3400
@@
 F 0 "Q5" H 5205 2204 50  0000 L CNN
 F 1 "Q_PMOS_DGS" H 5205 2295 50  0000 L CNN
-F 2 "" H 5200 2350 50  0001 C CNN
+F 2 "Package_TO_SOT_SMD:SOT-23" H 5200 2350 50  0001 C CNN
 F 3 "~" H 5000 2250 50  0001 C CNN
 	1    5000 2250
@@
 F 0 "Q4" H 4455 2004 50  0000 L CNN
 F 1 "Q_PMOS_DGS" H 4455 2095 50  0000 L CNN
-F 2 "" H 4450 2150 50  0001 C CNN
+F 2 "Package_TO_SOT_SMD:SOT-23" H 4450 2150 50  0001 C CNN
 F 3 "~" H 4250 2050 50  0001 C CNN
 	1    4250 2050
@@
 F 0 "Q6" H 5955 2354 50  0000 L CNN
 F 1 "Q_PMOS_DGS" H 5955 2445 50  0000 L CNN
-F 2 "" H 5950 2500 50  0001 C CNN
+F 2 "Package_TO_SOT_SMD:SOT-23" H 5950 2500 50  0001 C CNN
 F 3 "~" H 5750 2400 50  0001 C CNN
 	1    5750 2400
@@
 F 0 "R4" H 4220 2896 50  0000 L CNN
 F 1 "R" H 4220 2805 50  0000 L CNN
-F 2 "" V 4080 2850 50  0001 C CNN
+F 2 "Resistor_SMD:R_0603_1608Metric" V 4080 2850 50  0001 C CNN
 F 3 "~" H 4150 2850 50  0001 C CNN
 	1    4150 2850
@@
 F 0 "R5" H 4970 2896 50  0000 L CNN
 F 1 "R" H 4970 2805 50  0000 L CNN
-F 2 "" V 4830 2850 50  0001 C CNN
+F 2 "Resistor_SMD:R_0603_1608Metric" V 4830 2850 50  0001 C CNN
 F 3 "~" H 4900 2850 50  0001 C CNN
 	1    4900 2850
@@
 F 0 "R6" H 5720 2896 50  0000 L CNN
 F 1 "R" H 5720 2805 50  0000 L CNN
-F 2 "" V 5580 2850 50  0001 C CNN
+F 2 "Resistor_SMD:R_0603_1608Metric" V 5580 2850 50  0001 C CNN
 F 3 "~" H 5650 2850 50  0001 C CNN
 	1    5650 2850
