File: base_board/beer_mug.kicad_pcb (KiCad board)
At the start: 2 copper layers, 60.5 x 34 mm, 38 parts, among them J1 Conn_01x02, J2 Conn_01x02, J3 Conn_01x08, J4 Conn_01x02, J5 Conn_01x03, J6 Conn_01x02, Q1 Q_NMOS_DGS, Q2 Q_NMOS_DGS, Q3 Q_NMOS_DGS, Q4 Q_PMOS_DGS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

Commit message: pcb update
Connections:
- U3 pad 27: Net-(U3-Pad27) -> /Red
- U3 pad 28: /Red -> /Green
- U3 pad 29: /Green -> Net-(U3-Pad29)
Routing:
- net /Red: track 4.50 -> 2.66 mm
- net /Green: track 3.09 -> 4.28 mm
Changed lines of the file:
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@@
     (thickness 1.6)
     (drawings 2)
-    (tracks 210)
+    (tracks 208)
     (zones 0)
     (modules 38)
@@
   )
   (setup
-    (last_trace_width 0.5)
+    (last_trace_width 0.25)
     (user_trace_width 0.5)
     (trace_clearance 0.2)
@@
   (net 47 /A5)
   (net 48 "Net-(U3-Pad5)")
-  (net 49 "Net-(U3-Pad27)")
+  (net 49 "Net-(U3-Pad29)")
   (net_class Default "This is the default net class."
     (clearance 0.2)
@@
     (add_net "Net-(U3-Pad25)")
     (add_net "Net-(U3-Pad26)")
-    (add_net "Net-(U3-Pad27)")
+    (add_net "Net-(U3-Pad29)")
     (add_net "Net-(U3-Pad5)")
     (add_net "Net-(U3-Pad7)")
@@
       (net 19 /Blue))
     (pad 29 thru_hole circle (at -6.35 -7.62) (size 1.524 1.524) (drill 0.762) (layers *.Cu *.Mask)
+      (net 49 "Net-(U3-Pad29)"))
+    (pad 28 thru_hole circle (at -3.81 -7.62) (size 1.524 1.524) (drill 0.762) (layers *.Cu *.Mask)
       (net 18 /Green))
-    (pad 28 thru_hole circle (at -3.81 -7.62) (size 1.524 1.524) (drill 0.762) (layers *.Cu *.Mask)
+    (pad 27 thru_hole circle (at -1.27 -7.62) (size 1.524 1.524) (drill 0.762) (layers *.Cu *.Mask)
       (net 17 /Red))
-    (pad 27 thru_hole circle (at -1.27 -7.62) (size 1.524 1.524) (drill 0.762) (layers *.Cu *.Mask)
-      (net 49 "Net-(U3-Pad27)"))
     (pad 26 thru_hole circle (at 1.27 -7.62) (size 1.524 1.524) (drill 0.762) (layers *.Cu *.Mask)
       (net 32 "Net-(U3-Pad26)"))
@@
   (segment (start 77.825 51.635) (end 77.825 52.5) (width 0.25) (layer F.Cu) (net 16))
   (segment (start 81.22 48.24) (end 77.825 51.635) (width 0.25) (layer F.Cu) (net 16))
-  (segment (start 83.5 35.55) (end 83.05 35.55) (width 0.25) (layer B.Cu) (net 17))
-  (segment (start 81.22 34.22) (end 81.22 33) (width 0.25) (layer B.Cu) (net 17))
-  (segment (start 82.55 35.55) (end 81.22 34.22) (width 0.25) (layer B.Cu) (net 17))
-  (segment (start 82.55 35.55) (end 83.5 35.55) (width 0.25) (layer B.Cu) (net 17))
-  (segment (start 78.5 33.18) (end 78.68 33) (width 0.25) (layer B.Cu) (net 18))
-  (segment (start 78 33.68) (end 78.68 33) (width 0.25) (layer B.Cu) (net 18))
-  (segment (start 78 35.55) (end 78 33.68) (width 0.25) (layer B.Cu) (net 18))
+  (segment (start 83.5 33.26) (end 83.76 33) (width 0.25) (layer B.Cu) (net 17))
+  (segment (start 83.5 35.55) (end 83.5 33.26) (width 0.25) (layer B.Cu) (net 17))
+  (segment (start 78.67 35.55) (end 81.22 33) (width 0.25) (layer B.Cu) (net 18))
+  (segment (start 78 35.55) (end 78.67 35.55) (width 0.25) (layer B.Cu) (net 18))
+  (segment (start 78.5 33.18) (end 78.68 33) (width 0.25) (layer B.Cu) (net 49))
   (segment (start 74 35.14) (end 76.14 33) (width 0.25) (layer B.Cu) (net 19))
   (segment (start 73.59 35.55) (end 76.14 33) (width 0.25) (layer B.Cu) (net 19))
